Commit message: simplify r1 mesh for faster collision checking

File: mani_skill/assets/robots/galaxea_r1/r1_coacd.urdf (robot description, URDF)
Before this commit: robot R1, 30 links, 29 joints
Links:
- link base_link: geometry collision mesh filename=meshes_coacd/base_link.glb; visual mesh filename=meshes/base_link.STL
- link left_arm_link1: geometry collision mesh filename=meshes_coacd/left_arm_link1.glb; visual mesh filename=meshes/left_arm_link1.STL
- link left_arm_link2: geometry collision mesh filename=meshes_coacd/left_arm_link2.glb; visual mesh filename=meshes/left_arm_link2.STL
- link left_arm_link3: geometry collision mesh filename=meshes_coacd/left_arm_link3.glb; visual mesh filename=meshes/left_arm_link3.STL
- link left_arm_link4: geometry collision mesh filename=meshes_coacd/left_arm_link4.glb; visual mesh filename=meshes/left_arm_link4.STL
- link left_arm_link5: geometry collision mesh filename=meshes_coacd/left_arm_link5.glb; visual mesh filename=meshes/left_arm_link5.STL
- link left_arm_link6: geometry collision mesh filename=meshes_coacd/left_arm_link6.glb; visual mesh filename=meshes/left_arm_link6.STL
- link left_gripper_link1: geometry collision mesh filename=meshes_coacd/left_gripper_link1.glb; visual mesh filename=meshes/left_gripper_link1.STL
- link left_gripper_link2: geometry collision mesh filename=meshes_coacd/left_gripper_link2.glb; visual mesh filename=meshes/left_gripper_link2.STL
- link left_realsense_link: geometry collision mesh filename=meshes_coacd/left_realsense_link.glb; visual mesh filename=meshes/left_realsense_link.STL
- link right_arm_link1: geometry collision mesh filename=meshes_coacd/right_arm_link1.glb; visual mesh filename=meshes/right_arm_link1.STL
- link right_arm_link2: geometry collision mesh filename=meshes_coacd/right_arm_link2.glb; visual mesh filename=meshes/right_arm_link2.STL
- link right_arm_link3: geometry collision mesh filename=meshes_coacd/right_arm_link3.glb; visual mesh filename=meshes/right_arm_link3.STL
- link right_arm_link4: geometry collision mesh filename=meshes_coacd/right_arm_link4.glb; visual mesh filename=meshes/right_arm_link4.STL
- link right_arm_link5: geometry collision mesh filename=meshes_coacd/right_arm_link5.glb; visual mesh filename=meshes/right_arm_link5.STL
- link right_arm_link6: geometry collision mesh filename=meshes_coacd/right_arm_link6.glb; visual mesh filename=meshes/right_arm_link6.STL
- link right_gripper_link1: geometry collision mesh filename=meshes_coacd/right_gripper_link1.glb; visual mesh filename=meshes/right_gripper_link1.STL
- link right_gripper_link2: geometry collision mesh filename=meshes_coacd/right_gripper_link2.glb; visual mesh filename=meshes/right_gripper_link2.STL
- link right_realsense_link: geometry collision mesh filename=meshes_coacd/right_realsense_link.glb; visual mesh filename=meshes/right_realsense_link.STL
- link servo_link1: geometry collision mesh filename=meshes_coacd/servo_link1.glb; visual mesh filename=meshes/servo_link1.STL
- link servo_link2: geometry collision mesh filename=meshes_coacd/servo_link2.glb; visual mesh filename=meshes/servo_link2.STL
- link servo_link3: geometry collision mesh filename=meshes_coacd/servo_link3.glb; visual mesh filename=meshes/servo_link3.STL
- link torso_link1: geometry collision mesh filename=meshes_coacd/torso_link1.glb; visual mesh filename=meshes/torso_link1.STL
- link torso_link2: geometry collision mesh filename=meshes_coacd/torso_link2.glb; visual mesh filename=meshes/torso_link2.STL
- link torso_link3: geometry collision mesh filename=meshes_coacd/torso_link3.glb; visual mesh filename=meshes/torso_link3.STL
- link torso_link4: geometry collision mesh filename=meshes_coacd/torso_link4.glb; visual mesh filename=meshes/torso_link4.STL
- link wheel_link1: geometry collision mesh filename=meshes_coacd/wheel_link1.glb; visual mesh filename=meshes/wheel_link1.STL
- link wheel_link2: geometry collision mesh filename=meshes_coacd/wheel_link2.glb; visual mesh filename=meshes/wheel_link2.STL
- link wheel_link3: geometry collision mesh filename=meshes_coacd/wheel_link3.glb; visual mesh filename=meshes/wheel_link3.STL
- link zed_link: geometry collision mesh filename=meshes_coacd/zed_link.glb; visual mesh filename=meshes/zed_link.STL

File: mani_skill/assets/robots/galaxea_r1/r1_upperbody.urdf (robot description, URDF)
Before this commit: robot R1, 30 links, 29 joints
Joints:
- joint torso_joint1: type fixed -> revolute
- joint torso_joint2: type fixed -> revolute
- joint torso_joint3: type fixed -> revolute
- joint torso_joint4: type fixed -> revolute

File: mani_skill/assets/robots/galaxea_r1/r1_upperbody_coacd.urdf (robot description, URDF)
Before this commit: robot R1, 30 links, 29 joints
Links:
- link base_link: geometry collision mesh filename=meshes_coacd/base_link.glb; visual mesh filename=meshes/base_link.STL
- link left_arm_link1: geometry collision mesh filename=meshes_coacd/left_arm_link1.glb; visual mesh filename=meshes/left_arm_link1.STL
- link left_arm_link2: geometry collision mesh filename=meshes_coacd/left_arm_link2.glb; visual mesh filename=meshes/left_arm_link2.STL
- link left_arm_link3: geometry collision mesh filename=meshes_coacd/left_arm_link3.glb; visual mesh filename=meshes/left_arm_link3.STL
- link left_arm_link4: geometry collision mesh filename=meshes_coacd/left_arm_link4.glb; visual mesh filename=meshes/left_arm_link4.STL
- link left_arm_link5: geometry collision mesh filename=meshes_coacd/left_arm_link5.glb; visual mesh filename=meshes/left_arm_link5.STL
- link left_arm_link6: geometry collision mesh filename=meshes_coacd/left_arm_link6.glb; visual mesh filename=meshes/left_arm_link6.STL
- link left_gripper_link1: geometry collision mesh filename=meshes_coacd/left_gripper_link1.glb; visual mesh filename=meshes/left_gripper_link1.STL
- link left_gripper_link2: geometry collision mesh filename=meshes_coacd/left_gripper_link2.glb; visual mesh filename=meshes/left_gripper_link2.STL
- link left_realsense_link: geometry collision mesh filename=meshes_coacd/left_realsense_link.glb; visual mesh filename=meshes/left_realsense_link.STL
- link right_arm_link1: geometry collision mesh filename=meshes_coacd/right_arm_link1.glb; visual mesh filename=meshes/right_arm_link1.STL
- link right_arm_link2: geometry collision mesh filename=meshes_coacd/right_arm_link2.glb; visual mesh filename=meshes/right_arm_link2.STL
- link right_arm_link3: geometry collision mesh filename=meshes_coacd/right_arm_link3.glb; visual mesh filename=meshes/right_arm_link3.STL
- link right_arm_link4: geometry collision mesh filename=meshes_coacd/right_arm_link4.glb; visual mesh filename=meshes/right_arm_link4.STL
- link right_arm_link5: geometry collision mesh filename=meshes_coacd/right_arm_link5.glb; visual mesh filename=meshes/right_arm_link5.STL
- link right_arm_link6: geometry collision mesh filename=meshes_coacd/right_arm_link6.glb; visual mesh filename=meshes/right_arm_link6.STL
- link right_gripper_link1: geometry collision mesh filename=meshes_coacd/right_gripper_link1.glb; visual mesh filename=meshes/right_gripper_link1.STL
- link right_gripper_link2: geometry collision mesh filename=meshes_coacd/right_gripper_link2.glb; visual mesh filename=meshes/right_gripper_link2.STL
- link right_realsense_link: geometry collision mesh filename=meshes_coacd/right_realsense_link.glb; visual mesh filename=meshes/right_realsense_link.STL
- link servo_link1: geometry collision mesh filename=meshes_coacd/servo_link1.glb; visual mesh filename=meshes/servo_link1.STL
- link servo_link2: geometry collision mesh filename=meshes_coacd/servo_link2.glb; visual mesh filename=meshes/servo_link2.STL
- link servo_link3: geometry collision mesh filename=meshes_coacd/servo_link3.glb; visual mesh filename=meshes/servo_link3.STL
- link torso_link1: geometry collision mesh filename=meshes_coacd/torso_link1.glb; visual mesh filename=meshes/torso_link1.STL
- link torso_link2: geometry collision mesh filename=meshes_coacd/torso_link2.glb; visual mesh filename=meshes/torso_link2.STL
- link torso_link3: geometry collision mesh filename=meshes_coacd/torso_link3.glb; visual mesh filename=meshes/torso_link3.STL
- link torso_link4: geometry collision mesh filename=meshes_coacd/torso_link4.glb; visual mesh filename=meshes/torso_link4.STL
- link wheel_link1: geometry collision mesh filename=meshes_coacd/wheel_link1.glb; visual mesh filename=meshes/wheel_link1.STL
- link wheel_link2: geometry collision mesh filename=meshes_coacd/wheel_link2.glb; visual mesh filename=meshes/wheel_link2.STL
- link wheel_link3: geometry collision mesh filename=meshes_coacd/wheel_link3.glb; visual mesh filename=meshes/wheel_link3.STL
- link zed_link: geometry collision mesh filename=meshes_coacd/zed_link.glb; visual mesh filename=meshes/zed_link.STL
Joints:
- joint torso_joint1: type fixed -> revolute
- joint torso_joint2: type fixed -> revolute
- joint torso_joint3: type fixed -> revolute
- joint torso_joint4: type fixed -> revolute
